File: HDMI Breakout.kicad_sch (KiCad schematic)
At the start: 22 parts, among them J1 HC-HDMI0019T-1, J2 HC-HDMI0019T-1, U1 TMDS171IRGZT

Commit message: Before fixup2
Parts:
- added R19: 80.6 1%, Resistor_SMD:R_0402_1005Metric, symbol Device:R_US
- C10, C7: JLCPCB C1856484 -> C346216
- R1: value 7.06k 1% -> 6.98k 1%; JLCPCB C2500653 -> C4345381
Connections:
- net GND: now also R19.1; no longer R1.1
- new net: R1.1, R19.2
Other:
- moved on the sheet: R1
Changed lines of the file:
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@@
 	)
 	(junction
-		(at 161.29 151.13)
-		(diameter 0)
-		(color 0 0 0 0)
-	)
-	(junction
 		(at 340.36 24.13)
 		(diameter 0)
@@
 	)
 	(junction
+		(at 161.29 151.13)
+		(diameter 0)
+		(color 0 0 0 0)
+	)
+	(junction
 		(at 392.43 36.83)
 		(diameter 0)
@@
 	(wire
 		(pts
+			(xy 161.29 151.13) (xy 161.29 161.29)
+		)
+		(stroke
+			(width 0)
+			(type default)
+		)
+	)
+	(wire
+		(pts
 			(xy 171.45 128.27) (xy 189.23 128.27)
 		)
@@
 	(wire
 		(pts
-			(xy 181.61 151.13) (xy 189.23 151.13)
+			(xy 187.96 151.13) (xy 189.23 151.13)
 		)
 		(stroke
@@
 	(wire
 		(pts
-			(xy 161.29 151.13) (xy 161.29 161.29)
+			(xy 161.29 85.09) (xy 161.29 151.13)
 		)
 		(stroke
@@
 	(wire
 		(pts
-			(xy 149.86 158.75) (xy 149.86 161.29)
+			(xy 173.99 151.13) (xy 180.34 151.13)
 		)
 		(stroke
@@
 	(wire
 		(pts
-			(xy 54.61 106.68) (xy 68.58 106.68)
+			(xy 149.86 158.75) (xy 149.86 161.29)
 		)
 		(stroke
@@
 	(wire
 		(pts
-			(xy 340.36 24.13) (xy 353.06 24.13)
+			(xy 54.61 106.68) (xy 68.58 106.68)
 		)
 		(stroke
@@
 	(wire
 		(pts
-			(xy 170.18 69.85) (xy 189.23 69.85)
+			(xy 340.36 24.13) (xy 353.06 24.13)
 		)
 		(stroke
@@
 	(wire
 		(pts
-			(xy 54.61 101.6) (xy 68.58 101.6)
+			(xy 170.18 69.85) (xy 189.23 69.85)
 		)
 		(stroke
@@
 	(wire
 		(pts
-			(xy 326.39 24.13) (xy 326.39 26.67)
+			(xy 54.61 101.6) (xy 68.58 101.6)
 		)
 		(stroke
@@
 	(wire
 		(pts
-			(xy 340.36 59.69) (xy 340.36 62.23)
+			(xy 326.39 24.13) (xy 326.39 26.67)
 		)
 		(stroke
@@
 	(wire
 		(pts
-			(xy 161.29 151.13) (xy 173.99 151.13)
+			(xy 340.36 59.69) (xy 340.36 62.23)
 		)
 		(stroke
@@
 	(wire
 		(pts
-			(xy 36.83 144.78) (xy 36.83 146.05)
+			(xy 161.29 151.13) (xy 166.37 151.13)
 		)
 		(stroke
@@
 	(wire
 		(pts
-			(xy 161.29 85.09) (xy 161.29 151.13)
+			(xy 36.83 144.78) (xy 36.83 146.05)
 		)
 		(stroke
@@
 	)
 	(symbol
+		(lib_id "Device:R_US")
+		(at 170.18 151.13 90)
+		(unit 1)
+		(exclude_from_sim no)
+		(in_bom yes)
+		(on_board yes)
+		(dnp no)
+		(property "Reference" "R19"
+			(at 170.18 148.336 90)
+			(effects
+				(font
+					(size 1.27 1.27)
+				)
+			)
+		)
+		(property "Value" "80.6 1%"
+			(at 170.18 153.67 90)
+			(effects
+				(font
+					(size 1.27 1.27)
+				)
+			)
+		)
+		(property "Footprint" "Resistor_SMD:R_0402_1005Metric"
+			(at 170.434 150.114 90)
+			(effects
+				(font
+					(size 1.27 1.27)
+				)
+				(hide yes)
+			)
+		)
+		(property "Datasheet" "~"
+			(at 170.18 151.13 0)
+			(effects
+				(font
+					(size 1.27 1.27)
+				)
+				(hide yes)
+			)
+		)
+		(property "Description" "Resistor, US symbol"
+			(at 170.18 151.13 0)
+			(effects
+				(font
+					(size 1.27 1.27)
+				)
+				(hide yes)
+			)
+		)
+		(property "JLCPCB" ""
+			(at 170.434 156.718 90)
+			(show_name yes)
+			(effects
+				(font
+					(size 1.27 1.27)
+				)
+			)
+		)
+		(property "JCBPCB" ""
+			(at 170.18 151.13 0)
+			(effects
+				(font
+					(size 1.27 1.27)
+				)
+				(hide yes)
+			)
+		)
+		(pin "1"
+		)
+		(pin "2"
+		)
+		(instances
+			(project "HDMI Breakout"
+				(path "/7e1b48bc-ae7f-4b09-a989-3d4d32e543f0"
+					(reference "R19")
+					(unit 1)
+				)
+			)
+		)
+	)
+	(symbol
 		(lib_id "Device:C")
 		(at 378.46 30.48 0)
@@
 			)
 		)
-		(property "JLCPCB" "C1856484"
+		(property "JLCPCB" "C346216"
 			(at 406.4 39.37 0)
 			(show_name yes)
@@
 	(symbol
 		(lib_id "Device:R_US")
-		(at 177.8 151.13 90)
+		(at 184.15 151.13 90)
 		(unit 1)
 		(exclude_from_sim no)
@@
 		(dnp no)
 		(property "Reference" "R1"
-			(at 177.8 148.336 90)
+			(at 184.15 148.336 90)
 			(effects
 				(font
@@
 			)
 		)
-		(property "Value" "7.06k 1%"
-			(at 177.8 153.67 90)
+		(property "Value" "6.98k 1%"
+			(at 184.15 153.67 90)
 			(effects
 				(font
@@
 		)
 		(property "Footprint" "Resistor_SMD:R_0402_1005Metric"
-			(at 178.054 150.114 90)
+			(at 184.404 150.114 90)
 			(effects
 				(font
@@
 		)
 		(property "Datasheet" "~"
-			(at 177.8 151.13 0)
+			(at 184.15 151.13 0)
 			(effects
 				(font
@@
 		)
 		(property "Description" "Resistor, US symbol"
-			(at 177.8 151.13 0)
+			(at 184.15 151.13 0)
 			(effects
 				(font
@@
 			)
 		)
-		(property "JLCPCB" "C2500653"
-			(at 178.054 156.718 90)
+		(property "JLCPCB" "C4345381"
+			(at 184.404 156.718 90)
 			(show_name yes)
 			(effects
@@
 		)
 		(property "JCBPCB" ""
-			(at 177.8 151.13 0)
+			(at 184.15 151.13 0)
 			(effects
 				(font
@@
 			)
 		)
-		(property "JLCPCB" "C1856484"
+		(property "JLCPCB" "C346216"
 			(at 354.33 57.658 0)
 			(show_name yes)

Commit message: Update before DFM changes
Parts:
- C1, C14, C2, C3, C4, C8, C9: JLCPCB C1853272 -> C1525
- C10, C7: JLCPCB C346216 -> C5189822
- R1: JLCPCB C4345381 -> C47500
- R19: JLCPCB (none) -> C25134
Other:
- moved on the sheet: C14, R19
Changed lines of the file:
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@@
 	)
 	(junction
-		(at 161.29 161.29)
+		(at 157.48 161.29)
 		(diameter 0)
 		(color 0 0 0 0)
@@
 	)
 	(junction
-		(at 161.29 151.13)
-		(diameter 0)
-		(color 0 0 0 0)
-	)
-	(junction
 		(at 392.43 36.83)
 		(diameter 0)
@@
 	)
 	(junction
+		(at 157.48 151.13)
+		(diameter 0)
+		(color 0 0 0 0)
+	)
+	(junction
 		(at 326.39 24.13)
 		(diameter 0)
@@
 	)
 	(junction
-		(at 149.86 146.05)
+		(at 44.45 144.78)
 		(diameter 0)
 		(color 0 0 0 0)
 	)
 	(junction
-		(at 44.45 144.78)
+		(at 146.05 146.05)
 		(diameter 0)
 		(color 0 0 0 0)
@@
 	(wire
 		(pts
-			(xy 189.23 85.09) (xy 161.29 85.09)
+			(xy 189.23 85.09) (xy 157.48 85.09)
 		)
 		(stroke
@@
 	(wire
 		(pts
-			(xy 161.29 151.13) (xy 161.29 161.29)
+			(xy 157.48 151.13) (xy 157.48 161.29)
 		)
 		(stroke
@@
 	(wire
 		(pts
-			(xy 161.29 85.09) (xy 161.29 151.13)
+			(xy 157.48 85.09) (xy 157.48 151.13)
 		)
 		(stroke
@@
 	(wire
 		(pts
+			(xy 157.48 151.13) (xy 163.83 151.13)
+		)
+		(stroke
+			(width 0)
+			(type default)
+		)
+	)
+	(wire
+		(pts
 			(xy 118.11 100.33) (xy 189.23 100.33)
 		)
@@
 	(wire
 		(pts
-			(xy 118.11 146.05) (xy 149.86 146.05)
+			(xy 118.11 146.05) (xy 146.05 146.05)
+		)
+		(stroke
+			(width 0)
+			(type default)
+		)
+	)
+	(wire
+		(pts
+			(xy 146.05 146.05) (xy 189.23 146.05)
 		)
 		(stroke
@@
 	(wire
 		(pts
-			(xy 173.99 151.13) (xy 180.34 151.13)
+			(xy 171.45 151.13) (xy 180.34 151.13)
 		)
 		(stroke
@@
 	(wire
 		(pts
-			(xy 149.86 158.75) (xy 149.86 161.29)
+			(xy 146.05 158.75) (xy 146.05 161.29)
 		)
 		(stroke
@@
 	(wire
 		(pts
-			(xy 149.86 146.05) (xy 189.23 146.05)
-		)
-		(stroke
-			(width 0)
-			(type default)
-		)
-	)
-	(wire
-		(pts
 			(xy 240.03 77.47) (xy 270.51 77.47)
 		)
@@
 	(wire
 		(pts
-			(xy 149.86 146.05) (xy 149.86 151.13)
+			(xy 146.05 146.05) (xy 146.05 151.13)
 		)
 		(stroke
@@
 	(wire
 		(pts
-			(xy 161.29 151.13) (xy 166.37 151.13)
-		)
-		(stroke
-			(width 0)
-			(type default)
-		)
-	)
-	(wire
-		(pts
 			(xy 36.83 144.78) (xy 36.83 146.05)
 		)
@@
 	(wire
 		(pts
-			(xy 149.86 161.29) (xy 161.29 161.29)
+			(xy 146.05 161.29) (xy 157.48 161.29)
 		)
 		(stroke
@@
 	(wire
 		(pts
-			(xy 161.29 163.83) (xy 161.29 161.29)
+			(xy 157.48 163.83) (xy 157.48 161.29)
 		)
 		(stroke
@@
 	(symbol
 		(lib_id "Device:C")
-		(at 149.86 154.94 0)
+		(at 146.05 154.94 0)
 		(unit 1)
 		(exclude_from_sim no)
@@
 		(dnp no)
 		(property "Reference" "C14"
-			(at 153.67 153.6699 0)
+			(at 149.86 153.6699 0)
 			(effects
 				(font
@@
 		)
 		(property "Value" "0.1uF"
-			(at 153.67 156.2099 0)
+			(at 149.86 156.2099 0)
 			(effects
 				(font
@@
 		)
 		(property "Footprint" "Capacitor_SMD:C_0402_1005Metric"
-			(at 150.8252 158.75 0)
+			(at 147.0152 158.75 0)
 			(effects
 				(font
@@
 		)
 		(property "Datasheet" "~"
-			(at 149.86 154.94 0)
+			(at 146.05 154.94 0)
 			(effects
 				(font
@@
 		)
 		(property "Description" "Unpolarized capacitor"
-			(at 149.86 154.94 0)
+			(at 146.05 154.94 0)
 			(effects
 				(font
@@
 			)
 		)
-		(property "JLCPCB" "C1853272"
-			(at 136.652 154.94 0)
+		(property "JLCPCB" "C1525"
+			(at 132.842 154.94 0)
 			(show_name yes)
 			(effects
@@
 		)
 		(property "JCBPCB" ""
-			(at 149.86 154.94 0)
+			(at 146.05 154.94 0)
 			(effects
 				(font
@@
 			)
 		)
-		(property "JLCPCB" "C1853272"
+		(property "JLCPCB" "C1525"
 			(at 365.76 21.336 0)
 			(show_name yes)
@@
 			)
 		)
-		(property "JLCPCB" "C1853272"
+		(property "JLCPCB" "C1525"
 			(at 340.106 74.93 0)
 			(show_name yes)
@@
 			)
 		)
-		(property "JLCPCB" "C1853272"
+		(property "JLCPCB" "C1525"
 			(at 313.69 66.04 0)
 			(show_name yes)
@@
 	(symbol
 		(lib_id "Device:R_US")
-		(at 170.18 151.13 90)
+		(at 167.64 151.13 90)
 		(unit 1)
 		(exclude_from_sim no)
@@
 		(dnp no)
 		(property "Reference" "R19"
-			(at 170.18 148.336 90)
+			(at 167.64 148.336 90)
 			(effects
 				(font
@@
 		)
 		(property "Value" "80.6 1%"
-			(at 170.18 153.67 90)
+			(at 167.64 153.67 90)
 			(effects
 				(font
@@
 		)
 		(property "Footprint" "Resistor_SMD:R_0402_1005Metric"
-			(at 170.434 150.114 90)
+			(at 167.894 150.114 90)
 			(effects
 				(font
@@
 		)
 		(property "Datasheet" "~"
-			(at 170.18 151.13 0)
+			(at 167.64 151.13 0)
 			(effects
 				(font
@@
 		)
 		(property "Description" "Resistor, US symbol"
-			(at 170.18 151.13 0)
+			(at 167.64 151.13 0)
 			(effects
 				(font
@@
 			)
 		)
-		(property "JLCPCB" ""
-			(at 170.434 156.718 90)
+		(property "JLCPCB" "C25134"
+			(at 167.894 156.718 90)
 			(show_name yes)
 			(effects
@@
 		)
 		(property "JCBPCB" ""
-			(at 170.18 151.13 0)
+			(at 167.64 151.13 0)
 			(effects
 				(font
@@
 			)
 		)
-		(property "JLCPCB" "C1853272"
+		(property "JLCPCB" "C1525"
 			(at 340.36 21.336 0)
 			(show_name yes)
@@
 			)
 		)
-		(property "JLCPCB" "C1853272"
+		(property "JLCPCB" "C1525"
 			(at 314.198 30.48 0)
 			(show_name yes)
@@
 			)
 		)
-		(property "JLCPCB" "C346216"
+		(property "JLCPCB" "C5189822"
 			(at 406.4 39.37 0)
 			(show_name yes)
@@
 			)
 		)
-		(property "JLCPCB" "C4345381"
+		(property "JLCPCB" "C47500"
 			(at 184.404 156.718 90)
 			(show_name yes)
@@
 	(symbol
 		(lib_id "power:GND")
-		(at 161.29 163.83 0)
+		(at 157.48 163.83 0)
 		(unit 1)
 		(exclude_from_sim no)
@@
 		(fields_autoplaced yes)
 		(property "Reference" "#PWR09"
-			(at 161.29 170.18 0)
+			(at 157.48 170.18 0)
 			(effects
 				(font
@@
 		)
 		(property "Value" "GND"
-			(at 161.29 168.91 0)
+			(at 157.48 168.91 0)
 			(effects
 				(font
@@
 		)
 		(property "Footprint" ""
-			(at 161.29 163.83 0)
+			(at 157.48 163.83 0)
 			(effects
 				(font
@@
 		)
 		(property "Datasheet" ""
-			(at 161.29 163.83 0)
+			(at 157.48 163.83 0)
 			(effects
 				(font
@@
 		)
 		(property "Description" "Power symbol creates a global label with name \"GND\" , ground"
-			(at 161.29 163.83 0)
+			(at 157.48 163.83 0)
 			(effects
 				(font
@@
 			)
 		)
-		(property "JLCPCB" "C346216"
+		(property "JLCPCB" "C5189822"
 			(at 354.33 57.658 0)
 			(show_name yes)
@@
 			)
 		)
-		(property "JLCPCB" "C1853272"
+		(property "JLCPCB" "C1525"
 			(at 353.06 39.37 0)
 			(show_name yes)
