File: esp32.kicad_sch (KiCad schematic)
At the start: 43 parts, among them J3 HC-TYPE-C-16P-CH3.18-3A-02, J4 HC-TYPE-C-16P-CH3.18-3A-02, Q1 BC847BDW1T1G, SW1 B3FS-4055P, SW2 B3FS-4055P, U2 ESP32-C6-WROOM-1, U3 CP2102N-A02-GQFN28R

Commit message: Before fixup2
Parts:
- C11, C25, C28, C29: JLCPCB C1856484 -> C346216
- R11, R12, R13, R14: JLCPCB C4319604 -> C2131849
- R15, R16, R17, R18: JLCPCB C4112064 -> C2131941
- R6: JLCPCB C4231501 -> C2130243
- R7: JLCPCB C4351795 -> C4096848
Changed lines of the file:
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@@
 			)
 		)
-		(property "JLCPCB" "C4231501"
+		(property "JLCPCB" "C2130243"
 			(at 47.498 79.248 90)
 			(show_name yes)
@@
 			)
 		)
-		(property "JLCPCB" "C4351795"
+		(property "JLCPCB" "C4096848"
 			(at 50.8 92.71 90)
 			(show_name yes)
@@
 			)
 		)
-		(property "JLCPCB" "C4319604"
+		(property "JLCPCB" "C2131849"
 			(at 88.646 239.776 90)
 			(show_name yes)
@@
 			)
 		)
-		(property "JLCPCB" "C4319604"
+		(property "JLCPCB" "C2131849"
 			(at 69.85 180.34 90)
 			(show_name yes)
@@
 			)
 		)
-		(property "JLCPCB" "C4319604"
+		(property "JLCPCB" "C2131849"
 			(at 88.392 176.276 90)
 			(show_name yes)
@@
 			)
 		)
-		(property "JLCPCB" "C1856484"
+		(property "JLCPCB" "C346216"
 			(at 39.116 49.53 0)
 			(show_name yes)
@@
 			)
 		)
-		(property "JLCPCB" "C1856484"
+		(property "JLCPCB" "C346216"
 			(at 157.48 165.862 0)
 			(show_name yes)
@@
 			)
 		)
-		(property "JLCPCB" "C4112064"
+		(property "JLCPCB" "C2131941"
 			(at 288.544 173.99 0)
 			(show_name yes)
@@
 			)
 		)
-		(property "JLCPCB" "C4112064"
+		(property "JLCPCB" "C2131941"
 			(at 243.332 246.888 0)
 			(show_name yes)
@@
 			)
 		)
-		(property "JLCPCB" "C4319604"
+		(property "JLCPCB" "C2131849"
 			(at 69.596 244.094 90)
 			(show_name yes)
@@
 			)
 		)
-		(property "JLCPCB" "C1856484"
+		(property "JLCPCB" "C346216"
 			(at 197.866 31.75 0)
 			(show_name yes)
@@
 			)
 		)
-		(property "JLCPCB" "C4112064"
+		(property "JLCPCB" "C2131941"
 			(at 239.014 182.88 0)
 			(show_name yes)
@@
 			)
 		)
-		(property "JLCPCB" "C4112064"
+		(property "JLCPCB" "C2131941"
 			(at 288.544 212.09 0)
 			(show_name yes)
@@
 			)
 		)
-		(property "JLCPCB" "C1856484"
+		(property "JLCPCB" "C346216"
 			(at 157.48 229.362 0)
 			(show_name yes)

Commit message: Update before DFM changes
Parts:
- C11, C25, C28, C29: JLCPCB C346216 -> C5189822
- C12, C13, C26: JLCPCB C1853272 -> C1525
- C15, C27: JLCPCB C1852899 -> C14445
- R10, R2, R3, R4, R8: JLCPCB C4275117 -> C60490
- R11, R12, R13, R14: JLCPCB C2131849 -> C25905
- R15, R16, R17, R18: JLCPCB C2131941 -> C427206
- R5: JLCPCB C4161303 -> C25117
- R6: JLCPCB C2130243 -> C43473
- R7: JLCPCB C4096848 -> C25901
- R9: JLCPCB C6649868 -> C17168
Changed lines of the file:
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@@
 			)
 		)
-		(property "JLCPCB" "C2130243"
+		(property "JLCPCB" "C43473"
 			(at 47.498 79.248 90)
 			(show_name yes)
@@
 			)
 		)
-		(property "JLCPCB" "C4275117"
+		(property "JLCPCB" "C60490"
 			(at 135.89 117.856 90)
 			(show_name yes)
@@
 			)
 		)
-		(property "JLCPCB" "C1852899"
+		(property "JLCPCB" "C14445"
 			(at 75.438 92.964 0)
 			(show_name yes)
@@
 			)
 		)
-		(property "JLCPCB" "C4096848"
+		(property "JLCPCB" "C25901"
 			(at 50.8 92.71 90)
 			(show_name yes)
@@
 			)
 		)
-		(property "JLCPCB" "C2131849"
+		(property "JLCPCB" "C25905"
 			(at 88.646 239.776 90)
 			(show_name yes)
@@
 			)
 		)
-		(property "JLCPCB" "C2131849"
+		(property "JLCPCB" "C25905"
 			(at 69.85 180.34 90)
 			(show_name yes)
@@
 			)
 		)
-		(property "JLCPCB" "C4275117"
+		(property "JLCPCB" "C60490"
 			(at 68.326 53.34 90)
 			(show_name yes)
@@
 			)
 		)
-		(property "JLCPCB" "C4275117"
+		(property "JLCPCB" "C60490"
 			(at 330.962 121.92 0)
 			(show_name yes)
@@
 			)
 		)
-		(property "JLCPCB" "C2131849"
+		(property "JLCPCB" "C25905"
 			(at 88.392 176.276 90)
 			(show_name yes)
@@
 			)
 		)
-		(property "JLCPCB" "C346216"
+		(property "JLCPCB" "C5189822"
 			(at 39.116 49.53 0)
 			(show_name yes)
@@
 			)
 		)
-		(property "JLCPCB" "C346216"
+		(property "JLCPCB" "C5189822"
 			(at 157.48 165.862 0)
 			(show_name yes)
@@
 			)
 		)
-		(property "JLCPCB" "C1853272"
+		(property "JLCPCB" "C1525"
 			(at 322.072 88.9 0)
 			(show_name yes)
@@
 			)
 		)
-		(property "JLCPCB" "C6649868"
+		(property "JLCPCB" "C17168"
 			(at 330.708 111.506 0)
 			(show_name yes)
@@
 			)
 		)
-		(property "JLCPCB" "C2131941"
+		(property "JLCPCB" "C427206"
 			(at 288.544 173.99 0)
 			(show_name yes)
@@
 			)
 		)
-		(property "JLCPCB" "C2131941"
+		(property "JLCPCB" "C427206"
 			(at 243.332 246.888 0)
 			(show_name yes)
@@
 			)
 		)
-		(property "JLCPCB" "C4275117"
+		(property "JLCPCB" "C60490"
 			(at 371.856 52.07 90)
 			(show_name yes)
@@
 			)
 		)
-		(property "JLCPCB" "C1853272"
+		(property "JLCPCB" "C1525"
 			(at 243.078 31.496 0)
 			(show_name yes)
@@
 			)
 		)
-		(property "JLCPCB" "C2131849"
+		(property "JLCPCB" "C25905"
 			(at 69.596 244.094 90)
 			(show_name yes)
@@
 			)
 		)
-		(property "JLCPCB" "C4161303"
+		(property "JLCPCB" "C25117"
 			(at 143.51 66.548 90)
 			(show_name yes)
@@
 			)
 		)
-		(property "JLCPCB" "C346216"
+		(property "JLCPCB" "C5189822"
 			(at 197.866 31.75 0)
 			(show_name yes)
@@
 			)
 		)
-		(property "JLCPCB" "C2131941"
+		(property "JLCPCB" "C427206"
 			(at 239.014 182.88 0)
 			(show_name yes)
@@
 			)
 		)
-		(property "JLCPCB" "C2131941"
+		(property "JLCPCB" "C427206"
 			(at 288.544 212.09 0)
 			(show_name yes)
@@
 			)
 		)
-		(property "JLCPCB" "C1852899"
+		(property "JLCPCB" "C14445"
 			(at 329.692 135.89 0)
 			(show_name yes)
@@
 			)
 		)
-		(property "JLCPCB" "C346216"
+		(property "JLCPCB" "C5189822"
 			(at 157.48 229.362 0)
 			(show_name yes)
@@
 			)
 		)
-		(property "JLCPCB" "C4275117"
+		(property "JLCPCB" "C60490"
 			(at 371.856 67.31 90)
 			(show_name yes)
@@
 			)
 		)
-		(property "JLCPCB" "C1853272"
+		(property "JLCPCB" "C1525"
 			(at 371.602 88.9 0)
 			(show_name yes)
