File: power.kicad_sch (KiCad schematic)
At the start: 11 parts, among them U4 AP2114HA-1.2TRG1, U5 AP2114HA-3.3TRG1

Commit message: Before fixup2
Parts:
- C17, C19, C21, C24: JLCPCB C1856484 -> C346216
Changed lines of the file:
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@@
 			)
 		)
-		(property "JLCPCB" "C1856484"
+		(property "JLCPCB" "C346216"
 			(at 90.17 102.108 0)
 			(show_name yes)
@@
 			)
 		)
-		(property "JLCPCB" "C1856484"
+		(property "JLCPCB" "C346216"
 			(at 247.904 91.44 0)
 			(show_name yes)
@@
 			)
 		)
-		(property "JLCPCB" "C1856484"
+		(property "JLCPCB" "C346216"
 			(at 247.142 44.45 0)
 			(show_name yes)
@@
 			)
 		)
-		(property "JLCPCB" "C1856484"
+		(property "JLCPCB" "C346216"
 			(at 93.98 52.578 0)
 			(show_name yes)

Commit message: Update before DFM changes
Parts:
- removed U4: AP2114HA-1.2TRG1, Package_TO_SOT_SMD:SOT-223, symbol Diodes:AP2114HA-1.2TRG1
- removed U5: AP2114HA-3.3TRG1, Package_TO_SOT_SMD:SOT-223, symbol Diodes:AP2114HA-1.2TRG1
- added U4: AMS1117-1.2, Package_TO_SOT_SMD:SOT-223, symbol HDMI Breakout:AMS1117-1.2
- added U5: AMS1117-3.3, Package_TO_SOT_SMD:SOT-223, symbol HDMI Breakout:AMS1117-3.3
- C16, C18, C20, C22, C23: JLCPCB C1853272 -> C1525
- C17, C19, C21, C24: JLCPCB C346216 -> C5189822
Connections:
- net +1V2: now also U4.2 (VOUT)
- net +3V3: now also U5.2 (VOUT)
- net +5V: now also U4.3 (VIN), U5.3 (VIN)
- net GND: now also U4.1 (ADJ/GND), U5.1 (ADJ/GND)
- new net PAD_1V2: U4.4 (PAD)
- new net PAD_3V3: U5.4 (PAD)
