File: HDMI Breakout.kicad_pcb (KiCad board)
At the start: 4 copper layers, 70 x 70 mm, 76 parts, among them J1 HC-HDMI0019T-1, J2 HC-HDMI0019T-1, J3 HC-TYPE-C-16P-CH3.18-3A-02, J4 HC-TYPE-C-16P-CH3.18-3A-02, Q1 BC847BDW1T1G, SW1 B3FS-4055P, SW2 B3FS-4055P, U1 TMDS171IRGZT, U2 ESP32-C6-WROOM-1, U3 CP2102N-A02-GQFN28R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

Commit message: Before fixup2
Parts:
- added R19: 80.6 1%, Resistor_SMD:R_0402_1005Metric, F.Cu at (86.3, 76.7)
- R1: value 7.06k 1% -> 6.98k 1%
- moved J2 3.59 mm to (114.0, 69.2)
- moved J1 3.56 mm to (56.0, 69.2)
Connections:
- R1 pad 1: GND -> Net-(R1-Pad1)
Routing:
- net GND: track 132.7 -> 125.3 mm, vias 63 -> 64
- net /ESP32/UART_DN: track 18.7 -> 17.4 mm
- net Net-(R1-Pad1): track 0.00 -> 1.15 mm
- net /ESP32/UART_DP: track 15.6 -> 15.0 mm
- net /CEC_SRC: track 37.7 -> 37.1 mm

Commit message: Update before DFM changes
Parts:
- U4: value AP2114HA-1.2TRG1 -> AMS1117-1.2
- U5: value AP2114HA-3.3TRG1 -> AMS1117-3.3
- moved C23 2.32 mm to (63.3, 79.1)
- moved U5 0.85 mm to (68.7, 78.0)
- moved C24 0.81 mm to (63.0, 81.5)
Connections:
- U4 pad 1: +5V -> GND
- U4 pad 2: GND -> +1V2
- U4 pad 3: +1V2 -> +5V
- U4 pad 4: GND -> /Power/PAD_1V2
- U5 pad 1: +5V -> GND
- U5 pad 2: GND -> +3V3
- U5 pad 3: +3V3 -> +5V
- U5 pad 4: GND -> /Power/PAD_3V3
Routing:
- net +5V: track 24.8 -> 36.5 mm
- net +3V3: track 29.5 -> 37.5 mm, vias 10 -> 11
- net GND: track 125.3 -> 128.4 mm
- net +1V2: track 21.8 -> 22.4 mm
- added copper zone on F.Cu, net /Power/PAD_1V2
- added copper zone on F.Cu, net /Power/PAD_3V3
- removed copper zone on F.Cu, net GND

Commit message: Checkpointing before moving to 1206 components
Routing:
- net GND: track 128.4 -> 171.6 mm, vias 64 -> 57
- net /ESP32/USB_DN: track 22.5 -> 32.7 mm
- net VBUSA: track 40.6 -> 47.9 mm, vias 0 -> 3
- net /ESP32/USB_DP: track 23.5 -> 30.0 mm, vias 0 -> 2
- net /UTILITY_SNK: track 32.9 -> 26.8 mm
- net +3V3: track 37.5 -> 33.4 mm, vias 11 -> 13
- net /CEC_SNK: track 38.9 -> 34.9 mm
- net +1V2: track 22.4 -> 18.4 mm, vias 6 -> 7
- net /SCL_SRC: track 37.3 -> 41.1 mm
- net +5V: track 36.5 -> 40.3 mm, vias 7 -> 8
- net /SDA_SRC: track 36.0 -> 39.2 mm
- net Net-(J4-CC2): track 9.49 -> 6.50 mm, vias 2 -> 0
- net /SCL_CTL: track 25.7 -> 28.6 mm, vias 0 -> 2
- net /ESP32/EN: track 56.0 -> 58.5 mm
- net /ESP32/UART_DP: track 15.0 -> 17.5 mm, vias 3 -> 2
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Other:
- board text added: "HDMI Widget Rev B © 2024 Ionosphere LLC"
- board text removed: "HDMI Widget Rev A © 2024 Ionosphere LLC"
